File: duke_bme.kicad_sch (KiCad schematic)
At the start: 0 parts

Commit message: update sheet metadata
change from using text annotation tool in the sheet footers to defining
the sheet metadata using the Page Settings interface
Other:
- note removed: "00"
- note removed: "Duke BME Project Template"
- note removed: "Insert Date Here"
- company: (none) -> Mark Palmeri (Duke University)
- title: (none) -> BME Project Template
Changed lines of the file:
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@@
 (kicad_sch (version 20211123) (generator eeschema)
   (paper "A4")
-  (text "Insert Date Here" (at 207.01 194.31 0)
-    (effects (font (size 1.27 1.27)) (justify left bottom))
-  )
-  (text "Duke BME Project Template" (at 186.69 190.5 0)
-    (effects (font (size 1.27 1.27)) (justify left bottom))
-  )
-  (text "00" (at 269.24 194.31 0)
-    (effects (font (size 1.27 1.27)) (justify left bottom))
+  (title_block
+    (title "BME Project Template")
+    (date "2022-02-16")
+    (rev "01")
+    (company "Mark Palmeri (Duke University)")
   )
   (sheet_instances
